File: hardware/version1.0/useq1/useq1.kicad_pcb (KiCad board)
At the start: 2 copper layers, 40.6 x 108 mm, 172 parts, among them J1 Hanbo_USB_C_Receptacle_USB2.0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, J10 Out A2, J11 Out A3, J12 Out D1, J13 Out D2, J14 Out D3, J15 SWD, J2 Gate In 1, J3 Gate In 2, J4 CV In 1, J5 CV In 2, J6 Conn_01x02, J7 Conn_02x01, J8 Conn_02x01, J9 Out A1, Q1 MMBT3904, Q2 MMBT3904, SW1 SW_Push, SW2 SW_SPST, U1 TLV76733DRVR, U10 TL072, U11 W25Q128JVS, U12 CJ431 SOT-23, U2 TL072, U3 MCP6002-xMS, U4 TLV76733DRVR, U5 CJ431 SOT-23, U6 CJ431 SOT-23, U7 RP2040, U8 TL072, U9 TL072, Y1 YXC X322512MSB4SI

Commit message: drum models
Parts:
- moved D9 2.52 mm to (169.1, 89.0), turned to 90 degrees
- moved R6 2.25 mm to (157.2, 26.1)
- moved R3 0.95 mm to (157.9, 23.6)
Routing:
- net Net-(D9-A): track 4.80 -> 7.47 mm
- net Net-(J1-CC1): track 6.66 -> 7.96 mm
- net GND: track 48.6 -> 49.7 mm
- net Net-(J1-CC2): track 10.1 -> 11.1 mm
Changed lines of the file:
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@@
   )
   (footprint "Resistor_SMD:R_0402_1005Metric" (layer "F.Cu")
-    (at 158.8 23.25 180)
+    (at 157.92 23.62 180)
     (descr "Resistor SMD 0402 (1005 Metric), square (rectangular) end terminal, IPC_7351 nominal, (Body size source: IPC-SM-782 page 72, https://www.pcb-3d.com/wordpress/wp-content/uploads/ipc-sm-782a_amendment_1_and_2.pdf), generated with kicad-footprint-generator")
     (tags "resistor")
@@
   )
   (footprint "Resistor_SMD:R_0402_1005Metric" (layer "F.Cu")
-    (at 158.8 24.5 180)
+    (at 157.19 26.07 180)
     (descr "Resistor SMD 0402 (1005 Metric), square (rectangular) end terminal, IPC_7351 nominal, (Body size source: IPC-SM-782 page 72, https://www.pcb-3d.com/wordpress/wp-content/uploads/ipc-sm-782a_amendment_1_and_2.pdf), generated with kicad-footprint-generator")
     (tags "resistor")
@@
   )
   (footprint "LED_THT:LED_D3.0mm_FlatTop" (layer "B.Cu")
-    (at 169.1 86.525 -90)
+    (at 169.09 89.04 90)
     (descr "LED, Round, FlatTop, diameter 3.0mm, 2 pins, http://www.kingbright.com/attachments/file/psearch/000/00/00/L-47XEC(Ver.9A).pdf")
     (tags "LED Round FlatTop diameter 3.0mm 2 pins")
@@
     (fp_circle (center 1.27 0) (end 2.77 0)
       (stroke (width 0.1) (type solid)) (fill none) (layer "B.Fab"))
-    (pad "1" thru_hole rect (at 0 0 270) (size 1.8 1.8) (drill 0.9) (layers "*.Cu" "*.Mask")
+    (pad "1" thru_hole rect (at 0 0 90) (size 1.8 1.8) (drill 0.9) (layers "*.Cu" "*.Mask")
       (net 1 "GND") (pinfunction "K") (pintype "passive"))
-    (pad "2" thru_hole circle (at 2.54 0 270) (size 1.8 1.8) (drill 0.9) (layers "*.Cu" "*.Mask")
+    (pad "2" thru_hole circle (at 2.54 0 90) (size 1.8 1.8) (drill 0.9) (layers "*.Cu" "*.Mask")
       (net 30 "Net-(D9-A)") (pinfunction "A") (pintype "passive"))
     (model "${KICAD6_3DMODEL_DIR}/LED_THT.3dshapes/LED_D3.0mm_FlatTop.wrl"
@@
     (property "ki_description" "USB 2.0-only Type-C Receptacle connector")
     (property "ki_keywords" "usb universal serial bus type-C USB2.0")
-    (attr through_hole exclude_from_pos_files)
+    (attr through_hole)
     (fp_text reference "J1" (at 4.45 -3.875) (layer "B.SilkS")
         (effects (font (size 1.143 1.143) (thickness 0.152)) (justify left mirror))
@@
     (effects (font (size 0.2 0.2) (thickness 0.05)) (justify left bottom))
   )
+  (segment (start 156.68 26.07) (end 156.68 24.35) (width 0.3) (layer "F.Cu") (net 1))
   (segment (start 181.2 103.05) (end 180.25 104) (width 0.3) (layer "F.Cu") (net 1))
   (segment (start 167.2 43.85) (end 167.38775 43.85) (width 0.3) (layer "F.Cu") (net 1))
-  (segment (start 158.29 24.5) (end 158.29 23.25) (width 0.3) (layer "F.Cu") (net 1))
-  (segment (start 157.6 23.25) (end 156.75 22.4) (width 0.3) (layer "F.Cu") (net 1))
+  (segment (start 157.41 23.62) (end 156.75 22.96) (width 0.3) (layer "F.Cu") (net 1))
   (segment (start 163.05 52.8) (end 163.05 53.84) (width 0.3) (layer "F.Cu") (net 1))
   (segment (start 179.396946 35.2625) (end 179.2875 35.2625) (width 0.3) (layer "F.Cu") (net 1))
   (segment (start 160.02 35.15) (end 159.05 35.15) (width 0.5) (layer "F.Cu") (net 1))
   (segment (start 183 51.8) (end 183 54.872) (width 0.3) (layer "F.Cu") (net 1))
-  (segment (start 158.29 23.25) (end 157.6 23.25) (width 0.3) (layer "F.Cu") (net 1))
   (segment (start 179.2875 35.2625) (end 178.4 35.2625) (width 0.3) (layer "F.Cu") (net 1))
   (segment (start 180.248966 34.184312) (end 179.975 34.458278) (width 0.3) (layer "F.Cu") (net 1))
@@
   (segment (start 182.8625 44.975) (end 182.9 45.0125) (width 0.3) (layer "F.Cu") (net 1))
   (segment (start 168.35 53.25) (end 168.85 52.75) (width 0.3) (layer "F.Cu") (net 1))
+  (segment (start 156.68 24.35) (end 157.41 23.62) (width 0.3) (layer "F.Cu") (net 1))
   (segment (start 183 54.872) (end 183.318 55.19) (width 0.3) (layer "F.Cu") (net 1))
   (segment (start 153.525 37.65) (end 152.4 37.65) (width 0.3) (layer "F.Cu") (net 1))
@@
   (segment (start 154.5 31.655) (end 156.095 31.655) (width 0.3) (layer "F.Cu") (net 1))
   (segment (start 147.65 24.775) (end 148.175 24.775) (width 0.3) (layer "F.Cu") (net 1))
+  (segment (start 156.75 22.96) (end 156.75 22.4) (width 0.3) (layer "F.Cu") (net 1))
   (segment (start 165.65 53.84) (end 165.65 53.5) (width 0.3) (layer "F.Cu") (net 1))
   (segment (start 177.3375 67.075) (end 176.525001 67.075) (width 0.3) (layer "F.Cu") (net 1))
@@
   (segment (start 168.1 107.385) (end 169.1 108.385) (width 0.15) (layer "B.Cu") (net 29))
   (segment (start 168.1 106.4) (end 168.1 107.385) (width 0.15) (layer "B.Cu") (net 29))
-  (segment (start 168.1 93.45) (end 168.1 90.065) (width 0.15) (layer "F.Cu") (net 30))
-  (segment (start 168.1 90.065) (end 169.1 89.065) (width 0.15) (layer "F.Cu") (net 30))
+  (segment (start 168.1 93.45) (end 167.965 93.315) (width 0.15) (layer "F.Cu") (net 30))
+  (segment (start 167.965 93.315) (end 167.965 87.625) (width 0.15) (layer "F.Cu") (net 30))
+  (segment (start 167.965 87.625) (end 169.09 86.5) (width 0.15) (layer "F.Cu") (net 30))
   (segment (start 167.6 82.1) (end 167.6 77.1) (width 0.15) (layer "F.Cu") (net 31))
   (segment (start 167.6 77.1) (end 169.1 75.6) (width 0.15) (layer "F.Cu") (net 31))
@@
   (segment (start 176.714 32.076) (end 175.698 31.06) (width 1) (layer "B.Cu") (net 37))
   (segment (start 181.032 32.076) (end 176.714 32.076) (width 1) (layer "B.Cu") (net 37))
-  (segment (start 159.31 24.5) (end 160.465 25.655) (width 0.15) (layer "F.Cu") (net 38))
+  (segment (start 157.7 26.07) (end 158.115 25.655) (width 0.15) (layer "F.Cu") (net 38))
+  (segment (start 158.115 25.655) (end 163.47 25.655) (width 0.15) (layer "F.Cu") (net 38))
   (segment (start 163.47 25.655) (end 164.9 24.225) (width 0.15) (layer "F.Cu") (net 38))
-  (segment (start 160.465 25.655) (end 163.47 25.655) (width 0.15) (layer "F.Cu") (net 38))
   (segment (start 165.9 24.225) (end 165.9 23.930994) (width 0.73) (layer "F.Cu") (net 39))
   (segment (start 167.685 27.157254) (end 165.96 25.432254) (width 0.73) (layer "F.Cu") (net 39))
@@
   (segment (start 166.9 24.225) (end 166.9 23.869006) (width 0.73) (layer "B.Cu") (net 40))
   (segment (start 165.9 22.869006) (end 165.9 22.575) (width 0.73) (layer "B.Cu") (net 40))
-  (segment (start 159.31 23.25) (end 161.415 21.145) (width 0.15) (layer "F.Cu") (net 42))
+  (segment (start 161.245 21.145) (end 162.816726 21.145) (width 0.15) (layer "F.Cu") (net 42))
+  (segment (start 158.77 23.62) (end 161.245 21.145) (width 0.15) (layer "F.Cu") (net 42))
   (segment (start 162.816726 21.145) (end 163.271726 21.6) (width 0.15) (layer "F.Cu") (net 42))
-  (segment (start 161.415 21.145) (end 162.816726 21.145) (width 0.15) (layer "F.Cu") (net 42))
   (segment (start 163.271726 21.6) (end 166.925 21.6) (width 0.15) (layer "F.Cu") (net 42))
   (segment (start 166.925 21.6) (end 167.9 22.575) (width 0.15) (layer "F.Cu") (net 42))
+  (segment (start 158.43 23.62) (end 158.77 23.62) (width 0.15) (layer "F.Cu") (net 42))
   (segment (start 148.98 93.48) (end 148.85 93.35) (width 0.15) (layer "F.Cu") (net 44))
   (segment (start 149.7 93.48) (end 148.98 93.48) (width 0.15) (layer "F.Cu") (net 44))

Commit message: useq 1.0 hardware pinmap
Parts:
- removed J6: Conn_01x02, Connector_PinHeader_2.54mm:PinHeader_1x02_P2.54mm_Vertical
- added S2: B3U-1000P, digikey-footprints:Switch_Tactile_SMD_B3U-1000P, B.Cu at (148.5, 26.9)
- moved TP1 23.4 mm to (148.4, 21.7)
- moved FB2 10.8 mm to (184.9, 22.5), turned to -90 degrees
- moved D4 9.19 mm to (184.9, 26.1), turned to 90 degrees
- moved R3 5.45 mm to (152.7, 22.2)
- moved R6 5.18 mm to (152.7, 23.5)
- moved J1 3.54 mm to (162.9, 23.2)
- moved C3 3.36 mm to (184.0, 33.9)
- moved TP2 3.17 mm to (181.0, 45.2)
- moved SW2 2.77 mm to (178.3, 49.1)
- moved C5 2.57 mm to (182.9, 41.6)
- moved U4 2.57 mm to (180.5, 42.4)
- moved FB1 2.52 mm to (184.1, 36.7)
- moved C8 2.51 mm to (177.9, 43.0)
- moved C4 2.47 mm to (180.2, 38.8)
- moved D3 2.46 mm to (184.1, 38.8)
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Connections:
- net /GPIO1_LED_A3 renamed /GPIO11_LED_A3
- net /GPIO24_LED_CVIn1 renamed /GPIO24_LED_CVIn2
- net /GPIO25_LED_CVIn2 renamed /GPIO25_LED_CVIn1
- C34 pad 1: Net-(U8A--) -> Net-(U8A-+)
- C35 pad 1: Net-(U8B--) -> Net-(U8B-+)
- C36 pad 1: Net-(U9A--) -> Net-(U9A-+)
- R29 pad 2: /~{USB_BOOT} -> Net-(R29-Pad2)
- R41 pad 2: Net-(U8A--) -> Net-(U8A-+)
- R42 pad 2: Net-(U8B--) -> Net-(U8B-+)
- R43 pad 2: Net-(U9A--) -> Net-(U9A-+)
- R44 pad 2: Net-(U8A-+) -> Net-(U8A--)
- R45 pad 2: Net-(U8B-+) -> Net-(U8B--)
- R46 pad 2: Net-(U9A-+) -> Net-(U9A--)
- R47 pad 2: Net-(U10A-+) -> Net-(U10A--)
- R48 pad 2: Net-(U10B-+) -> Net-(U10B--)
- R49 pad 2: Net-(U9B-+) -> Net-(U9B--)
- R50 pad 2: Net-(U8A-+) -> Net-(U8A--)
- R51 pad 2: Net-(U8B-+) -> Net-(U8B--)
- R52 pad 2: Net-(U9A-+) -> Net-(U9A--)
- R53 pad 1: Net-(U8A-+) -> Net-(U8A--)
- R54 pad 1: Net-(U8B-+) -> Net-(U8B--)
- R55 pad 1: Net-(U9A-+) -> Net-(U9A--)
- R56 pad 1: Net-(U10A-+) -> Net-(U10A--)
- R57 pad 1: Net-(U10B-+) -> Net-(U10B--)
- R58 pad 1: Net-(U9B-+) -> Net-(U9B--)
- R7 pad 1: Net-(U2A-+) -> Net-(U2A--)
- R8 pad 1: Net-(U2B-+) -> Net-(U2B--)
- RV1 pad 3: Net-(U2A-+) -> Net-(U2A--)
- RV2 pad 3: Net-(U2B-+) -> Net-(U2B--)
- TP6 pad 1: Net-(U8A--) -> Net-(U8A-+)
- U10 pad 2: /GPIO18_Digital1 -> Net-(U10A--)
- U10 pad 3: Net-(U10A-+) -> /GPIO18_Digital1
- U10 pad 5: Net-(U10B-+) -> /GPIO17_Digital2
- U10 pad 6: /GPIO17_Digital2 -> Net-(U10B--)
- U2 pad 2: GND -> Net-(U2A--)
- U2 pad 3: Net-(U2A-+) -> GND
- U2 pad 5: Net-(U2B-+) -> GND
- U2 pad 6: GND -> Net-(U2B--)
- U9 pad 5: Net-(U9B-+) -> /GPIO16_Digital3
- U9 pad 6: /GPIO16_Digital3 -> Net-(U9B--)
Routing:
- net Net-(U9A-+): track 20.4 -> 81.5 mm
- net Net-(U8A--): track 78.3 -> 18.9 mm, vias 4 -> 0
- net Net-(U9A--): track 79.2 -> 20.6 mm
- net Net-(U8B--): track 77.5 -> 19.9 mm, vias 6 -> 0
- net Net-(U8B-+): track 22.4 -> 76.6 mm, vias 2 -> 4
- net Net-(U8A-+): track 19.3 -> 72.1 mm, vias 0 -> 4
- net Net-(U2B--): track 0.00 -> 28.1 mm, vias 0 -> 2
- net Net-(U2B-+): track 26.2 -> 0.00 mm, vias 2 -> 0
- net Net-(U9B-+): track 16.6 -> 0.00 mm
- net Net-(U2A-+): track 14.3 -> 0.00 mm, vias 2 -> 0
- net Net-(U2A--): track 0.00 -> 14.1 mm, vias 0 -> 2
- net Net-(U9B--): track 0.00 -> 12.1 mm
- net Net-(U10A--): track 0.00 -> 8.74 mm
- net +12V: track 232.1 -> 240.7 mm
- net Net-(U10A-+): track 7.73 -> 0.00 mm
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Other:
- board text added: "(version USEQ 1.0b) Emute Lab 2024"
- board text added: "GND"
- board text added: "SWCLK"
- board text added: "SWD"
- board text removed: "(version USEQ 1.0a) Emute Lab 2024"

Commit message: useq silkscreen updates
Other:
- board text added: "(version uSEQ 1.0b.b1) Emute Lab Instruments 2024"
- board text added: "RED"
- board text removed: "(version USEQ 1.0b) Emute Lab 2024"
- board text removed: "-12V STRIPE"

Commit message: i2c pullup fix
Connections:
- R31 pad 2: GND -> +3V3
- R37 pad 2: GND -> +3V3
Routing:
- net GND: track 42.1 -> 39.6 mm, vias 62 -> 61
- net +3V3: track 41.3 -> 42.7 mm
Other:
- board text added: "(version uSEQ 1.0c.b1) Emute Lab Instruments 2024"
- board text removed: "(version uSEQ 1.0b.b1) Emute Lab Instruments 2024"

Commit message: fixed editor cx issue, added analog ins, labelling on pcb
Routing:
- net Net-(R58-Pad2): track 39.7 -> 38.0 mm
- net +3V3: track 42.7 -> 41.3 mm
Other:
- board text added: "SCL"
- board text added: "SDA"
