File: hardware/version1.0/useq1/useq1.kicad_pcb (KiCad board)
At the start: 2 copper layers, 40.6 x 108 mm, 172 parts, among them J1 Hanbo_USB_C_Receptacle_USB2.0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, J10 Out A2, J11 Out A3, J12 Out D1, J13 Out D2, J14 Out D3, J15 SWD, J2 Gate In 1, J3 Gate In 2, J4 CV In 1, J5 CV In 2, J7 Conn_02x01, J8 Conn_02x01, J9 Out A1, Q1 MMBT3904, Q2 MMBT3904, SW1 SW_Push, SW2 SW_SPST, U1 TLV76733DRVR, U10 TL072, U11 W25Q128JVS, U12 CJ431 SOT-23, U2 TL072, U3 MCP6002-xMS, U4 TLV76733DRVR, U5 CJ431 SOT-23, U6 CJ431 SOT-23, U7 RP2040, U8 TL072, U9 TL072, Y1 YXC X322512MSB4SI

Commit message: 1.0c board edits
Parts:
- removed SW2: SW_SPST, benjiaomodular:ToggleSwitch_MTS-101_SPST
- added SW3: SW_SPDT, emutelab:Thonk DWB2, B.Cu at (183.5, 47.7)
- R23, R24, R25, R26, R27, R28, R32, R33, R34, R35, R65: value 820 -> 1.5k
- moved TP2 7.44 mm to (179.6, 52.5)
- moved TP5 1.71 mm to (177.8, 56.7)
Connections:
- U7 pad 35: /GPIO23 -> /GPIO23_SWTB
Routing:
- net /GPIO23_SWTB: track 0.00 -> 13.9 mm, vias 0 -> 1
- net /GPIO14_SWT: track 35.5 -> 46.7 mm, vias 1 -> 3
- net /GPIO22_LED_D3: track 95.6 -> 101.0 mm
- net /GPIO21_PWM1: track 17.7 -> 23.0 mm
- net /GPIO26_ADC0: track 43.8 -> 47.8 mm
- net GND: track 39.6 -> 35.7 mm, vias 61 -> 60
- net /RUN: track 56.4 -> 53.8 mm
- net /+3V3_SIG: track 45.2 -> 47.5 mm, vias 2 -> 3
- net /GPIO24_LED_CVIn2: track 72.5 -> 74.7 mm
- net /GPIO25_LED_CVIn1: track 55.1 -> 57.1 mm
- net /GPIO27_ADC1: track 46.2 -> 47.9 mm
- net Net-(J5-PadT): track 54.0 -> 53.1 mm
- net /GPIO20_PWM2: track 18.1 -> 18.8 mm, vias 0 -> 2

Commit message: hardware
Parts:
- R23, R24, R33, R34, R35: value 1.5k -> 18k
- R25, R26, R27, R28, R32: value 1.5k -> 9.1k
Routing:
- net GND: track 35.7 -> 38.7 mm, vias 60 -> 61
- net Net-(R11-Pad1): track 17.3 -> 17.8 mm
Other:
- board text added: "(version uSEQ 1.0c.b2) Emute Lab Instruments 2024"
- board text removed: "(version uSEQ 1.0c.b1) Emute Lab Instruments 2024"

Commit message: latest
Routing:
- net /GPIO4_LED_In2: track 75.1 -> 73.1 mm
- net /GPIO24_LED_CVIn2: track 74.9 -> 73.2 mm
- net Net-(U3B--): track 60.1 -> 59.2 mm
- net Net-(R11-Pad1): track 17.8 -> 17.0 mm
- net /GPIO8_GateInput1: track 45.7 -> 46.3 mm
