File: hardware/version1.0/useq1/useq1.kicad_pcb (KiCad board)
At the start: 2 copper layers, 40.6 x 108 mm, 172 parts, among them J1 Hanbo_USB_C_Receptacle_USB2.0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, J10 Out A2, J11 Out A3, J12 Out D1, J13 Out D2, J14 Out D3, J15 SWD, J2 Gate In 1, J3 Gate In 2, J4 CV In 1, J5 CV In 2, J7 Conn_02x01, J8 Conn_02x01, J9 Out A1, Q1 MMBT3904, Q2 MMBT3904, SW1 SW_Push, SW3 SW_SPDT, U1 TLV76733DRVR, U10 TL072, U11 W25Q128JVS, U12 CJ431 SOT-23, U2 TL072, U3 MCP6002-xMS, U4 TLV76733DRVR, U5 CJ431 SOT-23, U6 CJ431 SOT-23, U7 RP2040, U8 TL072, U9 TL072, Y1 YXC X322512MSB4SI

Commit message: 1.0d alpha hardware
Parts:
- R41, R42, R43: value 1.2k -> 10k
- moved R7 16.6 mm to (172.0, 54.5)
- moved R8 16.3 mm to (177.0, 59.1)
- moved C23 16.3 mm to (173.9, 60.1)
- moved U2 16.3 mm to (176.4, 55.7)
- moved C22 14.9 mm to (178.6, 52.2), turned to 0 degrees
- moved TP5 4.49 mm to (182.1, 57.8)
- moved TP2 3.38 mm to (182.0, 54.8)
- moved R2 1.99 mm to (153.9, 69.0)
- moved R11 1.10 mm to (175.9, 61.0)
Connections:
- R25 pad 1: /GPIO3_LED_A1 -> /GPIO14_LED_A1
- R27 pad 1: /GPIO24_LED_CVIn2 -> /GPIO6_LED_CVIn2
- R28 pad 1: /GPIO25_LED_CVIn1 -> /GPIO7_LED_CVIn1
- R65 pad 1: /GPIO6_LED_TEST -> /GPIO24_TEST_LED
- SW3 pad 1: /GPIO14_SWT -> /GPIO15_SWT
- U7 pad 17: /GPIO14_SWT -> /GPIO14_LED_A1
- U7 pad 18: /GPIO15 -> /GPIO15_SWT
- U7 pad 36: /GPIO24_LED_CVIn2 -> /GPIO24_TEST_LED
- U7 pad 37: /GPIO25_LED_CVIn1 -> /GPIO25
- U7 pad 5: /GPIO3_LED_A1 -> /GPIO3
- U7 pad 8: /GPIO6_LED_TEST -> /GPIO6_LED_CVIn2
- U7 pad 9: /GPIO7 -> /GPIO7_LED_CVIn1
Routing:
- net /GPIO6_LED_CVIn2: track 0.00 -> 85.8 mm, vias 0 -> 4
- net /GPIO3_LED_A1: track 84.5 -> 0.00 mm, vias 2 -> 0
- net /GPIO7_LED_CVIn1: track 0.00 -> 79.3 mm, vias 0 -> 8
- net /GPIO24_LED_CVIn2: track 73.2 -> 0.00 mm, vias 2 -> 0
- net /GPIO14_LED_A1: track 0.00 -> 63.9 mm
- net /GPIO25_LED_CVIn1: track 57.3 -> 0.00 mm, vias 4 -> 0
- net /GPIO14_SWT: track 46.7 -> 0.00 mm, vias 3 -> 0
- net /GPIO15_SWT: track 0.00 -> 33.6 mm, vias 0 -> 2
- net /GPIO24_TEST_LED: track 0.00 -> 31.6 mm, vias 0 -> 2
- net /GPIO6_LED_TEST: track 18.2 -> 0.00 mm, vias 2 -> 0
- net Net-(U2B--): track 28.1 -> 42.8 mm, vias 2 -> 4
- net +12V: track 240.7 -> 226.0 mm
- net Net-(R12-Pad1): track 11.5 -> 19.0 mm, vias 0 -> 2
- net Net-(U2A--): track 14.1 -> 21.6 mm, vias 2 -> 1
- net Net-(R11-Pad1): track 17.0 -> 9.83 mm
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Other:
- board text added: "(version uSEQ 1.0d) Emute Lab Instruments 2024"
- board text removed: "(version uSEQ 1.0c.b2) Emute Lab Instruments 2024"
