File: hardware/version1.0/useq1/useq1.kicad_sch (KiCad schematic)
At the start: 172 parts, among them J1 Hanbo_USB_C_Receptacle_USB2.0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, J10 Out A2, J11 Out A3, J12 Out D1, J13 Out D2, J14 Out D3, J15 SWD, J2 Gate In 1, J3 Gate In 2, J4 CV In 1, J5 CV In 2, J6 Conn_01x02, J7 Conn_02x01, J8 Conn_02x01, J9 Out A1, Q1 MMBT3904, Q2 MMBT3904, SW1 SW_Push, SW2 SW_SPST, U1 TLV76733DRVR, U10 TL072, U11 W25Q128JVS, U12 CJ431 SOT-23, U2 TL072, U3 MCP6002-xMS, U4 TLV76733DRVR, U5 CJ431 SOT-23, U6 CJ431 SOT-23, U7 RP2040, U8 TL072, U9 TL072, Y1 YXC X322512MSB4SI

Commit message: useq 1.0 hardware pinmap
Parts:
- removed J6: Conn_01x02, Connector_PinHeader_2.54mm:PinHeader_1x02_P2.54mm_Vertical, symbol Connector_Generic:Conn_01x02
- added S2: B3U-1000P, digikey-footprints:Switch_Tactile_SMD_B3U-1000P, symbol dk_Tactile-Switches:B3U-1000P
Connections:
- net GND: now also U2.3 (+), U2.5 (+), S2.1; no longer U2.2 (-), U2.6 (-)
- net GPIO16_Digital3: now also U9.5 (+); no longer U9.6 (-)
- net GPIO17_Digital2: now also U10.5 (+); no longer U10.6 (-)
- net GPIO18_Digital1: now also U10.3 (+); no longer U10.2 (-)
- net at R47.2, R56.1: now also U10.2 (-); no longer U10.3 (+)
- net at R44.2, R50.2, R53.1: now also U8.2 (-); no longer U8.3 (+)
- net at R46.2, R52.2, R55.1: now also U9.2 (-); no longer U9.3 (+)
- net at C35.1, R42.2: now also U8.5 (+); no longer U8.6 (-)
- net at R48.2, R57.1: now also U10.6 (-); no longer U10.5 (+)
- net at R8.1, RV2.3: now also U2.6 (-); no longer U2.5 (+)
- net at R49.2, R58.1: now also U9.6 (-); no longer U9.5 (+)
- net at C34.1, R41.2, TP6.1: now also U8.3 (+); no longer U8.2 (-)
- net at R45.2, R51.2, R54.1: now also U8.6 (-); no longer U8.5 (+)
- net at C36.1, R43.2: now also U9.3 (+); no longer U9.2 (-)
- net at R7.1, RV1.3: now also U2.2 (-); no longer U2.3 (+)
- net GPIO1_LED_A3 renamed GPIO11_LED_A3
- net GPIO24_LED_CVIn1 renamed GPIO24_LED_CVIn2
- net GPIO25_LED_CVIn2 renamed GPIO25_LED_CVIn1
- net ~{USB_BOOT}: no longer names the net of R29.2
- net ~{USB_BOOT}: now also S2.2
Other:
- note added: "https://modwiggler.com/forum/viewtopic.php?t=253062 https://electronotes.netfirms.com/AN235.pdf"

Commit message: i2c pullup fix
Connections:
- net +3V3: now also R31.2, R37.2
- net GND: no longer R31.2, R37.2
Changed lines of the file:
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@@
     )
   )
+  (symbol (lib_id "power:+3V3") (at 422.91 48.514 180) (unit 1)
+    (in_bom yes) (on_board yes) (dnp no) (fields_autoplaced)
+    (property "Reference" "#PWR058" (at 422.91 44.704 0)
+      (effects (font (size 1.27 1.27)) hide)
+    )
+    (property "Value" "+3V3" (at 422.91 52.6471 0)
+      (effects (font (size 1.27 1.27)))
+    )
+    (property "Footprint" "" (at 422.91 48.514 0)
+      (effects (font (size 1.27 1.27)) hide)
+    )
+    (property "Datasheet" "" (at 422.91 48.514 0)
+      (effects (font (size 1.27 1.27)) hide)
+    )
+    (pin "1")
+    (instances
+      (project "useq1"
+        (path "/7d928d56-093a-4ca8-aed1-414b7e703b45"
+          (reference "#PWR058") (unit 1)
+        )
+      )
+    )
+  )
   (symbol (lib_id "power:GND") (at 376.047 363.474 0) (unit 1)
     (in_bom yes) (on_board yes) (dnp no) (fields_autoplaced)
@@
     )
   )
-  (symbol (lib_id "power:GND") (at 435.61 48.514 0) (unit 1)
-    (in_bom yes) (on_board yes) (dnp no) (fields_autoplaced)
-    (property "Reference" "#PWR078" (at 435.61 54.864 0)
-      (effects (font (size 1.27 1.27)) hide)
-    )
-    (property "Value" "GND" (at 435.61 52.6471 0)
-      (effects (font (size 1.27 1.27)))
-    )
-    (property "Footprint" "" (at 435.61 48.514 0)
-      (effects (font (size 1.27 1.27)) hide)
-    )
-    (property "Datasheet" "" (at 435.61 48.514 0)
-      (effects (font (size 1.27 1.27)) hide)
-    )
-    (pin "1")
-    (instances
-      (project "useq1"
-        (path "/7d928d56-093a-4ca8-aed1-414b7e703b45"
-          (reference "#PWR078") (unit 1)
-        )
-      )
-    )
-  )
   (symbol (lib_id "Device:C") (at 339.09 182.372 0) (unit 1)
     (in_bom yes) (on_board yes) (dnp no) (fields_autoplaced)
@@
     )
   )
-  (symbol (lib_id "power:GND") (at 422.91 48.514 0) (unit 1)
-    (in_bom yes) (on_board yes) (dnp no) (fields_autoplaced)
-    (property "Reference" "#PWR074" (at 422.91 54.864 0)
-      (effects (font (size 1.27 1.27)) hide)
-    )
-    (property "Value" "GND" (at 422.91 52.6471 0)
-      (effects (font (size 1.27 1.27)))
-    )
-    (property "Footprint" "" (at 422.91 48.514 0)
-      (effects (font (size 1.27 1.27)) hide)
-    )
-    (property "Datasheet" "" (at 422.91 48.514 0)
-      (effects (font (size 1.27 1.27)) hide)
-    )
-    (pin "1")
-    (instances
-      (project "useq1"
-        (path "/7d928d56-093a-4ca8-aed1-414b7e703b45"
-          (reference "#PWR074") (unit 1)
-        )
-      )
-    )
-  )
   (symbol (lib_id "Amplifier_Operational:TL072") (at 83.82 174.371 0) (mirror x) (unit 1)
     (in_bom yes) (on_board yes) (dnp no)
@@
         )
       )
+    )
+  )
+  (symbol (lib_id "power:+3V3") (at 435.61 48.514 180) (unit 1)
+    (in_bom yes) (on_board yes) (dnp no) (fields_autoplaced)
+    (property "Reference" "#PWR074" (at 435.61 44.704 0)
+      (effects (font (size 1.27 1.27)) hide)
+    )
+    (property "Value" "+3V3" (at 435.61 52.6471 0)
+      (effects (font (size 1.27 1.27)))
+    )
+    (property "Footprint" "" (at 435.61 48.514 0)
+      (effects (font (size 1.27 1.27)) hide)
+    )
+    (property "Datasheet" "" (at 435.61 48.514 0)
+      (effects (font (size 1.27 1.27)) hide)
+    )
+    (pin "1")
+    (instances
+      (project "useq1"
+        (path "/7d928d56-093a-4ca8-aed1-414b7e703b45"
+          (reference "#PWR074") (unit 1)
+        )
+      )

Commit message: 1.0c board edits
Parts:
- removed SW2: SW_SPST, benjiaomodular:ToggleSwitch_MTS-101_SPST, symbol Switch:SW_SPST
- added SW3: SW_SPDT, emutelab:Thonk DWB2, symbol Switch:SW_SPDT
- R23, R24, R25, R26, R27, R28, R32, R33, R34, R35, R65: value 820 -> 1.5k
Connections:
- net GND: now also SW3.2 (B)
- net GPIO14_SWT: now also SW3.1 (A)
- net GPIO23 renamed GPIO23_SWTB
- net GPIO23_SWTB: now also SW3.3 (C)
Changed lines of the file:
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@@
     (effects (font (size 1.27 1.27)) (justify left bottom))
   )
-  (label "GPIO23" (at 292.1 286.512 180) (fields_autoplaced)
+  (label "GPIO23_SWTB" (at 292.1 286.512 180) (fields_autoplaced)
     (effects (font (size 1.27 1.27)) (justify right bottom))
   )
@@
     (effects (font (size 1.27 1.27)) (justify left bottom))
   )
+  (label "GPIO14_SWT" (at 144.018 93.98 0) (fields_autoplaced)
+    (effects (font (size 1.27 1.27)) (justify left bottom))
+  )
   (label "GPIO2_LED_A2" (at 348.234 105.283 0) (fields_autoplaced)
     (effects (font (size 1.27 1.27)) (justify left bottom))
@@
     (effects (font (size 1.27 1.27)) (justify right bottom))
   )
-  (label "GPIO14_SWT" (at 48.387 118.745 0) (fields_autoplaced)
-    (effects (font (size 1.27 1.27)) (justify left bottom))
-  )
   (label "GPIO18_Digital1" (at 473.329 235.839 0) (fields_autoplaced)
     (effects (font (size 1.27 1.27)) (justify left bottom))
@@
     (effects (font (size 1.27 1.27)) (justify right bottom))
   )
+  (label "GPIO23_SWTB" (at 144.018 99.06 0) (fields_autoplaced)
+    (effects (font (size 1.27 1.27)) (justify left bottom))
+  )
   (label "RUN" (at 51.816 135.382 0) (fields_autoplaced)
     (effects (font (size 1.27 1.27)) (justify left bottom))
@@
       (effects (font (size 1.27 1.27)))
     )
-    (property "Value" "820" (at 372.999 119.9459 90)
+    (property "Value" "1.5k" (at 372.999 119.9459 90)
       (effects (font (size 1.27 1.27)))
     )
@@
       (effects (font (size 1.27 1.27)))
     )
-    (property "Value" "820" (at 426.339 93.6569 90)
+    (property "Value" "1.5k" (at 426.339 93.6569 90)
       (effects (font (size 1.27 1.27)))
     )
@@
       (effects (font (size 1.27 1.27)))
     )
-    (property "Value" "820" (at 369.443 102.5469 90)
+    (property "Value" "1.5k" (at 369.443 102.5469 90)
       (effects (font (size 1.27 1.27)))
     )
@@
       (effects (font (size 1.27 1.27)))
     )
-    (property "Value" "820" (at 369.443 93.4029 90)
+    (property "Value" "1.5k" (at 369.443 93.4029 90)
       (effects (font (size 1.27 1.27)))
     )
@@
     )
   )
+  (symbol (lib_id "Switch:SW_SPDT") (at 138.938 96.52 0) (unit 1)
+    (in_bom yes) (on_board yes) (dnp no) (fields_autoplaced)
+    (property "Reference" "SW3" (at 138.938 88.6927 0)
+      (effects (font (size 1.27 1.27)))
+    )
+    (property "Value" "SW_SPDT" (at 138.938 91.1169 0)
+      (effects (font (size 1.27 1.27)))
+    )
+    (property "Footprint" "emutelab:Thonk DWB2" (at 138.938 96.52 0)
+      (effects (font (size 1.27 1.27)) hide)
+    )
+    (property "Datasheet" "~" (at 138.938 104.14 0)
+      (effects (font (size 1.27 1.27)) hide)
+    )
+    (pin "2")
+    (pin "1")
+    (pin "3")
+    (instances
+      (project "useq1"
+        (path "/7d928d56-093a-4ca8-aed1-414b7e703b45"
+          (reference "SW3") (unit 1)
+        )
+      )
+    )
+  )
   (symbol (lib_id "power:GND") (at 486.918 155.956 270) (unit 1)
     (in_bom yes) (on_board yes) (dnp no) (fields_autoplaced)
@@
       (effects (font (size 1.27 1.27)))
     )
-    (property "Value" "820" (at 426.339 75.3689 90)
+    (property "Value" "1.5k" (at 426.339 75.3689 90)
       (effects (font (size 1.27 1.27)))
     )
@@
     )
   )
-  (symbol (lib_id "power:GND") (at 38.227 118.745 0) (unit 1)
-    (in_bom yes) (on_board yes) (dnp no) (fields_autoplaced)
-    (property "Reference" "#PWR03" (at 38.227 125.095 0)
-      (effects (font (size 1.27 1.27)) hide)
-    )
-    (property "Value" "GND" (at 38.227 122.8781 0)
-      (effects (font (size 1.27 1.27)))
-    )
-    (property "Footprint" "" (at 38.227 118.745 0)
-      (effects (font (size 1.27 1.27)) hide)
-    )
-    (property "Datasheet" "" (at 38.227 118.745 0)
-      (effects (font (size 1.27 1.27)) hide)
-    )
-    (pin "1")
-    (instances
-      (project "useq1"
-        (path "/7d928d56-093a-4ca8-aed1-414b7e703b45"
-          (reference "#PWR03") (unit 1)
-        )
-      )
-    )
-  )
   (symbol (lib_id "Device:LED") (at 380.619 131.826 180) (unit 1)
     (in_bom yes) (on_board yes) (dnp no) (fields_autoplaced)
@@
     )
   )
-  (symbol (lib_id "Switch:SW_SPST") (at 43.307 118.745 0) (unit 1)
-    (in_bom yes) (on_board yes) (dnp no) (fields_autoplaced)
-    (property "Reference" "SW2" (at 43.307 112.9497 0)
-      (effects (font (size 1.27 1.27)))
-    )
-    (property "Value" "SW_SPST" (at 43.307 115.3739 0)
-      (effects (font (size 1.27 1.27)))
-    )
-    (property "Footprint" "benjiaomodular:ToggleSwitch_MTS-101_SPST" (at 43.307 118.745 0)
-      (effects (font (size 1.27 1.27)) hide)
-    )
-    (property "Datasheet" "~" (at 43.307 118.745 0)
-      (effects (font (size 1.27 1.27)) hide)
-    )
-    (pin "1")
-    (pin "2")
-    (instances
-      (project "useq1"
-        (path "/7d928d56-093a-4ca8-aed1-414b7e703b45"
-          (reference "SW2") (unit 1)
-        )
-      )
-    )
-  )
   (symbol (lib_id "Amplifier_Operational:TL072") (at 518.16 168.402 0) (mirror x) (unit 1)
     (in_bom yes) (on_board yes) (dnp no)
@@
     )
   )
+  (symbol (lib_id "power:GND") (at 133.858 96.52 270) (unit 1)
+    (in_bom yes) (on_board yes) (dnp no) (fields_autoplaced)
+    (property "Reference" "#PWR078" (at 127.508 96.52 0)
+      (effects (font (size 1.27 1.27)) hide)
+    )
+    (property "Value" "GND" (at 130.6831 96.52 90)
+      (effects (font (size 1.27 1.27)) (justify right))
+    )
+    (property "Footprint" "" (at 133.858 96.52 0)
+      (effects (font (size 1.27 1.27)) hide)
+    )
+    (property "Datasheet" "" (at 133.858 96.52 0)
+      (effects (font (size 1.27 1.27)) hide)
+    )
+    (pin "1")
+    (instances
+      (project "useq1"
+        (path "/7d928d56-093a-4ca8-aed1-414b7e703b45"
+          (reference "#PWR078") (unit 1)
+        )
+      )
+    )
+  )
   (symbol (lib_id "power:+12V") (at 91.44 379.73 0) (unit 1)
     (in_bom yes) (on_board yes) (dnp no) (fields_autoplaced)
@@
       (effects (font (size 1.27 1.27)))
     )
-    (property "Value" "820" (at 429.895 127.1849 90)
+    (property "Value" "1.5k" (at 429.895 127.1849 90)
       (effects (font (size 1.27 1.27)))
     )
@@
       (effects (font (size 1.27 1.27)))
     )
-    (property "Value" "820" (at 369.443 75.1149 90)
+    (property "Value" "1.5k" (at 369.443 75.1149 90)
       (effects (font (size 1.27 1.27)))
     )
@@
       (effects (font (size 1.27 1.27)))
     )
-    (property "Value" "820" (at 369.443 84.2589 90)
+    (property "Value" "1.5k" (at 369.443 84.2589 90)
       (effects (font (size 1.27 1.27)))
     )
@@
       (effects (font (size 1.27 1.27)))
     )
-    (property "Value" "820" (at 426.339 84.5129 90)
+    (property "Value" "1.5k" (at 426.339 84.5129 90)
       (effects (font (size 1.27 1.27)))
     )
@@
       (effects (font (size 1.27 1.27)))
     )
-    (property "Value" "820" (at 372.999 129.0899 90)
+    (property "Value" "1.5k" (at 372.999 129.0899 90)
       (effects (font (size 1.27 1.27)))
     )
@@
       (effects (font (size 1.27 1.27)))
     )
-    (property "Value" "820" (at 426.339 102.8009 90)
+    (property "Value" "1.5k" (at 426.339 102.8009 90)
       (effects (font (size 1.27 1.27)))
     )

Commit message: hardware
Parts:
- R23, R24, R33, R34, R35: value 1.5k -> 18k
- R25, R26, R27, R28, R32: value 1.5k -> 9.1k
Changed lines of the file:
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@@
       (effects (font (size 1.27 1.27)))
     )
-    (property "Value" "1.5k" (at 372.999 119.9459 90)
+    (property "Value" "9.1k" (at 372.999 119.9459 90)
       (effects (font (size 1.27 1.27)))
     )
@@
       (effects (font (size 1.27 1.27)))
     )
-    (property "Value" "1.5k" (at 426.339 93.6569 90)
+    (property "Value" "18k" (at 426.339 93.6569 90)
       (effects (font (size 1.27 1.27)))
     )
@@
       (effects (font (size 1.27 1.27)))
     )
-    (property "Value" "1.5k" (at 369.443 102.5469 90)
+    (property "Value" "9.1k" (at 369.443 102.5469 90)
       (effects (font (size 1.27 1.27)))
     )
@@
       (effects (font (size 1.27 1.27)))
     )
-    (property "Value" "1.5k" (at 369.443 93.4029 90)
+    (property "Value" "9.1k" (at 369.443 93.4029 90)
       (effects (font (size 1.27 1.27)))
     )
@@
       (effects (font (size 1.27 1.27)))
     )
-    (property "Value" "1.5k" (at 426.339 75.3689 90)
+    (property "Value" "9.1k" (at 426.339 75.3689 90)
       (effects (font (size 1.27 1.27)))
     )
@@
       (effects (font (size 1.27 1.27)))
     )
-    (property "Value" "1.5k" (at 369.443 75.1149 90)
+    (property "Value" "18k" (at 369.443 75.1149 90)
       (effects (font (size 1.27 1.27)))
     )
@@
       (effects (font (size 1.27 1.27)))
     )
-    (property "Value" "1.5k" (at 369.443 84.2589 90)
+    (property "Value" "18k" (at 369.443 84.2589 90)
       (effects (font (size 1.27 1.27)))
     )
@@
       (effects (font (size 1.27 1.27)))
     )
-    (property "Value" "1.5k" (at 426.339 84.5129 90)
+    (property "Value" "18k" (at 426.339 84.5129 90)
       (effects (font (size 1.27 1.27)))
     )
@@
       (effects (font (size 1.27 1.27)))
     )
-    (property "Value" "1.5k" (at 372.999 129.0899 90)
+    (property "Value" "9.1k" (at 372.999 129.0899 90)
       (effects (font (size 1.27 1.27)))
     )
@@
       (effects (font (size 1.27 1.27)))
     )
-    (property "Value" "1.5k" (at 426.339 102.8009 90)
+    (property "Value" "18k" (at 426.339 102.8009 90)
       (effects (font (size 1.27 1.27)))
     )

Commit message: latest
Parts:
- R41, R42, R43: value 1.2k -> 10k
Changed lines of the file:
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@@
     (effects (font (size 1.27 1.27)) (justify left top) (href "https://www.falstad.com/circuit/circuitjs.html?ctz=CQAgjCAMB0l3BWcZYA4BsB2ATNzZsEBOVA9EBSCkAFgGYKBTAWjDACgAnCzc9GkOlSpBAqjUzx2Ad0HDRckQRGQuPclQS8F4yXDVa+Amvx0g6dKQHNzqAaYtGoUGYvDYRvJR5c1IDSQFmOmwQVBDzUM0AfX5oyGiaDExosASYeEgiXgR0QmjWaOxohGi6V0MFSrYotRN7ATo7MwIpACV1cBpjVCowbucIP3BodCQUMecYBHYaNJBWcjAiUIjl0LTCEAA-ABUAGXoISAAdAGdh7HOwFgJzmEwQoiIabOw0iSIwBHuQK7PsLd-sxsNAEGBwnRntg6Ag5p8aL9TmcwOcQWCIRZobD4ZgXvdoI9sM9XjgPnjvtc-OdtgAXAA2R0YABNmABHAB20RZUHOIV6vIBfioyJwcEFFmgFmlMtl5H+KEBrH+D3e-QhOCIkGJvBVf3OoJoQLRGXgdHQQgQUNheDm5r1yNRZ2Yprg5st1oQtrA9oJZPVqE12uyeSpyLpjLoN1ZnO5rIAgorBRDoBC06QM+n9QDoNhMvn83RjWcYFhwgRcsTIBr8SXszRoMKC-mbsqCdWcFCkjh6KgXnQJEjru2wJ2XoHsL3+4OS6NMOXCHktTXESjqWcI0yY1yWcx46CoudeiLzpdrsWHsHiLDLH3J1pfv8lXdnYbsua4BC71qiD86460TfR50E-YQVh-P9L2Ja8rUgO8aAfNdwwZLd2R3ZlBSbTCqAVC9CX8L4QneEIkknJ0cINYsXVTfw6EkPBUAQDAwDGd4hxRE0aIsej5yY9AWK9cj8KhH1cFE0i5jDGkUKjXdYx5ZEBX+BBbjoP083QL47EDD5iVXCiUSoh50BI0lCF6EJtXYp1qN4Uy3iY-w8xVQkNK07tdNrfpkMjaM0LjPdpkFJTzzbZ1L0sSBHJvegvnI7MizC104NefpJwsb5tTyVB2NYdt4DsL4aHSqNKGwbLOMkSLoqtWK2HOEDpN8uSAAc42CgzWxfWztQsL0sBhSRiEwR8+WLUF52Kn1eDGXpoNyp0JrsYiZsc+bwvwmEbQGuiouyBqfNQtk2oUo9xUU87T06vD8FwJ5MC9R5ttGgEqLoMEmkyyB+Iyx5A2stF3qtUhKG+n0oz+kbZ1umEdUevryqkjcZL8+SMMdShguzFSksJLQ6O6AgVkY3ocrrXDWBshtypMDAJCaFYPDJk8OOdan+CEfg-sZ4Q-XxzBCeJDxHLJ7ymqO9C9yQR1Mmw7MuuBFBqxIKarU0gWmhe59FYxQNGKyLwyTmC9kzRFBwT1ygQwndUqKV5Zlu+c1sl7JHN1k7d2v+d2-OZdqZfFb2Ud3P2eQp+qziBz7J2+hBYLYWsDOfGyYDSPr+ieZITIwe41BY5BQmYIglgIZw830WR85YvoS9qDoi9rhZ+gEYuploPooimME1Fb3AW8bvpMh7+VJxAXv5EHqRK8b1uahcae-nkceVHYGx86Z8ByEcKYKm0TRtGYJJ586Q+lAPo-VEr8+z4H1wj77seR7EdgOjmLfmks2wxD+duRkmCZpZQG7twboIhLCNCEOYSA38vhTwoCBKBAhchUBtMfAa5hIEPVWJA1QNhzRgOgZEFBhCRSuHQeAwQOAMEr24MgxBlDVgkNoHoVQABDeBKDIHkMgd4JuGwCxtzSEPK+jdRxLD3uwdh1QfBCG8CIXhypwACNTn4R4CF9YOzxEQIB3lZH8D7G8C0AslFDz8AwVgAxFhN3IBfZAsQaDRBSD6cE+BUjpFgBWAoYBUjxFgFCb6hBXCz1LmIguvh-AgECH8XIYQIifxwugex8RUg4jwG43xmQQyVlKIUYo5Uyh33zk0JBCDinhIYM3duOEqH1DLnQJJCRnGjm8aUZKWS8g5O8Xk+p5RZCgPoXQihqgAD2Y8zB+GeNQNpOQOllzGeUIAA"))
   )
-  (text_box "lpf 13.2kHz\n"
+  (text_box "lpf 1.5kHz\n"
     (at 487.045 161.671 0) (size 21.844 23.114)
     (stroke (width 0) (type default))
@@
     (effects (font (size 1.27 1.27)) (justify left top) (href "https://www.falstad.com/circuit/circuitjs.html?ctz=CQAgjCAMB0l3BWcZYA4BsB2ATNzZsEBOVA9EBSCkAFgGYKBTAWjDACgAnCzc9GkOlSpBAqjUzx2Ad0HDRckQRGQuPclQS8F4yXDVa+Amvx0g6dKQHNzqAaYtGoUGYvDYRvJR5c1IDSQFmOmwQVBDzUM0AfX5oyGiaDExosASYeEgiXgR0QmjWaOxohGi6V0MFSrYotRN7ATo7MwIpACV1cBpjVCowbucIP3BodCQUMecYBHYaNJBWcjAiUIjl0LTCEAA-ABUAGXoISAAdAGdh7HOwFgJzmEwQoiIk9GfNzCI6e5Ars+xbn9mNhoAgwOE6Ag8BhDGwfqczmBzsDQeCLFDMDDeHCzg8ni8MO9IHgvtc-OdtgAXAA2R0YABNmABHAB20QZUHOIV6nP+fioCJwcF5FmgFnFEsl5D+KABrD+D2wbDmmAQcyIYHQllQPz+IJogORGXgdHQQihhDAuTG4JM8OuRtgJrNqAtYOtYLs6Hu0BwyrAqvVmu1ZIRVNpdBujNZ7MZAEFZbzwdBwanSOm079ziDsJk83m6IbcaNMZHLRDwardecaNB+fm8zd5T7IAHsH4mpWEL1TTrcUmW22O+nVT2hD6sOECJ6LF3QxSaXTo2yGcw4zneb0BTWqDKiw9iURu3R6HRskISNX-kWUTRspDUNghJGtKT+wikWdb-fu0+p6-vmLSRsCPcJT3PVBL0RckznDJdmRXeleXrZDd2ufdfX8DVcEgV08hWZ4rzlO4vxgNILEwT4YWJSAtQQQDt0RR1yLoSiSDGGi6IYzCzwIXM8JAkCiHnWDF0jVcYw5BEeT+BBbm4oU3gDEJc0jIgzSvJsSOYB48inPJVSaSEEHtJjSN9PTIwM+jwgQEygNzJTHhwtSNOgsMxKjBDYzXaZNzQxEbwPSxIAkF5TRPXgGKzM5C2bYtMjsDUsksEIaEIXJMFM1gW3gJK0i+fx2wyrBHUkEKwvoLUJC1c50A8iMvKZAAHWN-JirSgQPbALBVLCeySK84pIkFMRMXN3js4k72yz9Rq9CaNSm9thPM4DeoDfr-EGs56oXRqJNaqTzi3fzGMudD4oeAhNXoR4bQkDAiJvOhQSaOz0p6-B8DAVjTM-YI3tdNVcFYgM2D+oCbv4VjTTBR7vXc-b4MkpCP0oTcYrkq7fS0WjUEorQ0nozTbgB2snzvR9hEgTFnmJf7kQp-gSA8Xo6aIBmgLxoRCfwSASaR0SDuXHy4yQD9MlQjqbxQGjLUPbtnPHfs9RvVAUxPJpc1yR9IWyfcBy-DXfvoR8BaEHriEwWXYFzBWQKVkIVf6BqUcQmK4PExl6TayXhT+L2vN9jk91YT9XpsqFH3U0cafsgLiIBsj-H1-pbsVlZ7jUTVkFCZh1Lz5xc30WRc81PolgIFwOgLqv8-6ARC4FWg+iiKZQTUQvcCb+vBkyLvpXbEBu-kPoB7LvvC5qFxJ9+eRR5UdgbFztnwHIRwpgqbRNG0Zgklnzp96UPeD9UMvT5Pvvz9oEQe5HoexAqerfmGXI+hWGvaFzppGlzWwxDgFbiMSYEwJZQE7twboIhLCNCEOYUKgwS433fgggQqDIS1FkFgVY8DVS4KXjYXsaDIhUFgVvbgGDEHQJIWQkKqhKEv3bJoF+5DdBSGwTgEhODzDwIYRQVhiCeFsNoHoVQABDARZD4HCPgd4BY1c0h5hGIQVi41TRjSVFqFR9FHhzFdATeioUlh5lcAGPu5jwA7zMdoSxaoBCWJQQMOxL9HHPz6NoVB6wXCSOqD4IQ3gRDyPlOAfMvw6yhWII+N4-A2B2CQPqYxSoMqlgFhAJRUgOwKIGIsBR5Az7IFiDQaIKRfpgnwKkdIsBpwFDAKkeIsAzy0UIK4aeijbHV34XMDezQwSrGaOPfQABjCg1df6jNCPQduTYlDQFUXo8ESsjEmAgXADgNg+m0AiJsmhAoKhjN6awgZsx-AgECL8XIYQIghBbngIp8RUiQnSqUqpmRzy5HyIUYodzygAHsR5mD8M8agxo4DvLyOA0IRBzDsCAA"))
   )
-  (text_box "lpf 13.2kHz\n"
+  (text_box "lpf 10kHz\n"
     (at 486.791 105.029 0) (size 21.844 23.114)
     (stroke (width 0) (type default))
@@
     (effects (font (size 1.27 1.27)) (justify left top))
   )
-  (text_box "lpf 13.2kHz\n"
+  (text_box "lpf 1.5kHz\n"
     (at 486.664 49.022 0) (size 21.844 23.114)
     (stroke (width 0) (type default))
@@
       (effects (font (size 1.27 1.27)))
     )
-    (property "Value" "1.2k" (at 491.49 111.5639 90)
+    (property "Value" "10k" (at 491.49 111.5639 90)
       (effects (font (size 1.27 1.27)))
     )
@@
       (effects (font (size 1.27 1.27)))
     )
-    (property "Value" "1.2k" (at 491.363 55.5569 90)
+    (property "Value" "10k" (at 491.363 55.5569 90)
       (effects (font (size 1.27 1.27)))
     )
@@
       (effects (font (size 1.27 1.27)))
     )
-    (property "Value" "1.2k" (at 491.744 168.2059 90)
+    (property "Value" "10k" (at 491.744 168.2059 90)
       (effects (font (size 1.27 1.27)))
     )

Commit message: 1.0d alpha hardware
Connections:
- net GPIO14_SWT renamed GPIO14_LED_A1
- net GPIO14_LED_A1: now also R25.1; no longer SW3.1 (A)
- net GPIO15 renamed GPIO15_SWT
- net GPIO15_SWT: now also SW3.1 (A)
- net GPIO24_LED_CVIn2 renamed GPIO24_TEST_LED
- net GPIO24_TEST_LED: now also R65.1; no longer R27.1
- net GPIO25_LED_CVIn1 renamed GPIO25
- net GPIO25: no longer R28.1
- net GPIO3_LED_A1 renamed GPIO3
- net GPIO3: no longer R25.1
- net GPIO6_LED_TEST renamed GPIO6_LED_CVIn2
- net GPIO6_LED_CVIn2: now also R27.1; no longer R65.1
- net GPIO7 renamed GPIO7_LED_CVIn1
- net GPIO7_LED_CVIn1: now also R28.1
