File: hardware/version1.0/fr4panel/fr4panel/fr4panel.kicad_pcb (KiCad board)
At the start: 2 copper layers, 40.6 x 128.5 mm, 30 parts

Commit message: useq 1.0 hardware pinmap
Parts:
- added REF**: MountingHole_3mm, MountingHole:MountingHole_3mm, F.Cu at (162.1, 39.1)
- moved REF** 3.61 mm to (147.8, 30.9)
- moved REF** 2.74 mm to (132.2, 61.2)
Routing:
- added copper zone on F.Cu, net (none)
Other:
- board text added: "Prototype 1.0b"
- board text added: "USEQ"
- board text added: "bsel"
- board text added: "reset"
- board text removed: "USEQ Prototype 1.0a"

Commit message: 1.0c board edits
Parts:
- REF**: value PanelHole_ToggleSwitch_MTS-101 -> PanelHole_ToggleSwitch_Dailywell_DWB2; footprint benjiaomodular:PanelHole_ToggleSwitch_MTS-101 -> emutelab:PanelHole_ToggleSwitch_Dailywell_DWB2
- moved REF** 1.61 mm to (131.8, 59.7)
Other:
- board text added: "Prototype 1.0c"
- board text added: "uSEQ"
- board text removed: "Prototype 1.0b"
- board text removed: "USEQ"
